Commit message: Controller changes

File: xacro/OmuniRobot.xacro (robot description, xacro)
@@ -18,5 +18,5 @@
 			<child  link="${prefix}_link"/>
 			<insert_block name="joint_axis"/>
-		</joint>
+		</joint><!--
 		<transmission name="${prefix}_trans">
 			<type>transmission_interface/SimpleTransmission</type>
@@ -26,4 +26,14 @@
 			<actuator name="${prefix}_motor">
 				<hardwareInterface>hardware_interface/EffortJointInterface</hardwareInterface>
+				<mechanismReduction>1</mechanismReduction>
+			</actuator>
+		</transmission>-->
+		<transmission name="${prefix}_trans">
+			<type>transmission_interface/SimpleTransmission</type>
+			<joint name="${prefix}_joint">
+				<hardwareInterface>hardware_interface/VelocityJointInterface</hardwareInterface>
+			</joint>
+			<actuator name="${prefix}_motor">
+				<hardwareInterface>hardware_interface/VelocityJointInterface</hardwareInterface>
 				<mechanismReduction>1</mechanismReduction>
 			</actuator>
@@ -105,16 +115,16 @@
 	<gazebo>
 		<plugin name="gazebo_ros_control" filename="libgazebo_ros_control.so">
-		<robotNamespace>/OmuniRobot</robotNamespace>
-		<!--
-		<robotSimType>gazebo_ros_control/DefaultRobotHWSim</robotSimType>-->
-		<legacyModeNS>true</legacyModeNS>
+			<robotNamespace>/OmuniRobot</robotNamespace>
+			<!--
+			<robotSimType>gazebo_ros_control/DefaultRobotHWSim</robotSimType>-->
+			<legacyModeNS>true</legacyModeNS>
 		</plugin>
 	</gazebo>
 	<gazebo>
 		<plugin name="ground_truth" filename="libgazebo_ros_p3d.so">
-		<frameName>world</frameName>
-		<bodyName>base_link</bodyName>
-		<topicName>/tracker</topicName>
-		<updateRate>10.0</updateRate>
+			<frameName>world</frameName>
+			<bodyName>base_link</bodyName>
+			<topicName>/tracker</topicName>
+			<updateRate>10.0</updateRate>
 		</plugin>
 	</gazebo>

Commit message: Adjusting gmapping

File: xacro/OmuniRobot.xacro (robot description, xacro)
@@ -90,5 +90,5 @@
 			<origin xyz="0 0 0.03" rpy="0 0 0" />
 			<geometry>
-				<box size="0.20 0.20 0.05" />
+				<box size="0.20 0.20 0.04" />
 			</geometry>
 		</collision>
